File: wearable_cape.sch (KiCad schematic (older format))
At the start: 86 parts, among them J1 JACK_3P, J2 JACK_3P, J3 JACK_3P, P1 BELA_AINS, P2 RECEIVER, P3 BATTERY, P4 BELA_AOUTS, P5 PWR_OUT, P6 CONN_01X05, P7 CONN_01X05, SW1 SW_HALT, SW2 SW_MODE_SEL, SW3 SWITCH_SPDT, U1 MCP6004, U2 MCP6004, U3 BEAGLEBONEBLACK, U4 OKI_7805

Commit message: latest
Parts:
- C1, C10, C11, C14, C15, C16, C17, C2, C20, C23, C24, C3, C4, C5, C8, C9: symbol C -> Device:C
- C12, C13, C18, C19, C21, C22, C6, C7: symbol CP1 -> Device:CP1
- D1: symbol RG_Led -> wearable_cape:RG_Led
- FB1, FB2: symbol FILTER -> wearable_cape-rescue:FILTER
- J1, J2, J3: symbol JACK_3P -> jack_3p:JACK_3P
- P1: symbol BELA_AINS -> wearable_cape:BELA_AINS
- P2: symbol CONN_02X04 -> wearable_cape-rescue:CONN_02X04
- P3, P5: symbol CONN_01X02 -> wearable_cape:CONN_01X02
- P4: symbol BELA_AOUTS -> wearable_cape:BELA_AOUTS
- P6, P7: symbol CONN_01X05 -> wearable_cape-rescue:CONN_01X05
- R1, R10, R11, R12, R13, R14, R15, R16, R17, R18, R19, R2, R20, R21, R22, R23, R24, R25, R26, R27, R28, R29, R3, R30, R31, R32, R33, R34, R35, R36, R37, R38, R39, R4, R40, R41, R42, R5, R6, R7, R8, R9: symbol R -> Device:R
- SW1, SW2: symbol SW_PUSH -> wearable_cape:SW_PUSH
- SW3: symbol SWITCH_SPDT -> wearable_cape:SWITCH_SPDT
- U1, U2: symbol MCP6004 -> wearable_cape:MCP6004
- U3: symbol BEAGLEBONEBLACK -> beagleboneblack:BEAGLEBONEBLACK
- U4: symbol OKI_7805 -> oki_7805:OKI_7805
Connections:
- wire segments 283 -> 341
Other:
- note added: "NOTE: This resistor is not populated\non all filter circuits in production. \nIt was there for... what (??? - impedence matching?)\nmaybe its understandable for the audio capelet..\ndoes this help get better high freq response?\n\nIn the next version it will be removed."
- note added: "NOTE: This stage of each filter circuit \nwas left unpopulated on production boards. \nThe reasoning for this stage was to accommodate\ndifferent possible input impedences on amplifiers,\ninstead we assume the output goes to the input stage\nof one of the Adafruit MAX9744 boards and uses its input \nimpedence. The Adafruit boards have AC coupling caps\nat the input.. they could also be DC coupled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"
- note added: "Replace with \nvoltage reference"
